File: hardware/Rev1_00-0a/Consolation_Kicad/USB3.kicad_sch (KiCad schematic)
At the start: 13 parts, among them J1 0484050003, U3 AP2192AFGEG-7

Commit message: Update schematics, block diagram and pin mux (good progress G)
Parts:
- removed R143: 10K, footprint:RES_0402, symbol KicadCompDb:Resistors/RES_SMT_00013
- removed R58: 0R, footprint:RES_0603, symbol KicadCompDb:Resistors/RES_SMT_00021
- added C52: 47u, footprint:CAP_NONPOL_1206, symbol KicadCompDb:Capacitors/CAP_CER_SMT_00010
Connections:
- net CGND is gone; now on net GND: J1.10 (CGND), J1.11 (CGND)
- net CM5_USB3_VBUS_EN: now also U3.4 (EN2)
- net GND: now also C52.1
- net USB3_0.USB_VBUS: now also C52.2
- net RP2350_USB_VBUS: now reaches U3.6 (OUT2)
- no-connect marks 1 -> 0
Other:
- moved on the sheet: C46, C47, C49, C51, F1, R142, R146, R147, U3
