File: hardware/Rev1_00-0a/Consolation_Kicad/Consolation_Kicad.kicad_pcb (KiCad board)
At the start: 6 copper layers, 137.5 x 76.6 mm, 449 parts, among them J1 BM04B-SURS-TF, J10 61300311121, J11 5051102291, J12 RPI_CMx_B, J13 5051102291, J14 61300311121, J15 61300311121, J17 61300311121, J18 61300411121, J19 RPI_CMx_A, J2 SJ-3524-SMT-TR, J3 62684-402100ALF, J4 12401598E4#2A, J5 S2B-PH-K-S, J6 2086581001, J7 2998TR, J8 DM3AT-SF-PEJM5, Q1 SSM3K56FS,LF, Q10 SSM3K56FS,LF, Q11 SSM3K56FS,LF, Q12 SSM3K56FS,LF, Q14 SSM3K56FS,LF, Q18 SSM3K56FS,LF, Q19 SSM3K56FS,LF, Q20 SSM3K56FS,LF, Q21 SSM3K56FS,LF, Q22 SSM3K56FS,LF, Q23 SSM3K56FS,LF, Q24 SSM3K56FS,LF, Q25 SSM3K56FS,LF, Q26 SSM3K56FS,LF, Q27 SSM3K56FS,LF, Q28 SSM3K56FS,LF, Q29 SSM3K56FS,LF, Q3 SSM3K56FS,LF, Q7 SSM3K56FS,LF, Q8 SSM3K56FS,LF, Q9 SSM3K56FS,LF, U1 BQ25640VDLR, U10 TPS62826DMQR, U11 AP22913W6-7, U15 SN65DSI84ZXHR, U18 AP22913W6-7, U19 SN74LVC1G125DBVR, U2 RP2350A, U21 MCP7940NT-I/MS, U26 TPS61169DCKR, U30 STM6710DWB6F, U31 SN74LVC1G125DBVR, U32 SN74HCS365QPWRQ1, U4 ECS-2016MVQ-120-BP-TR, U5 NAU88C22YG, U6 AP22913W6-7, U7 TPS79901DRVR, U8 GD25Q32CWIGR, U9 TPS61230ARNSR, Y1 12MHz 10pF, Y2 32.768kHz

Commit message: Add teardrops, clean ERC and DRC check. Review design rules Update fill zones Add stitching vias
Routing:
- net /CODEC/LSPKOUT: track 95.1 -> 105.3 mm
- net GND: track 387.1 -> 378.0 mm, vias 495 -> 682
- net /CM5_CONN_B/USB2_RP2350.USB_P: track 54.5 -> 52.7 mm
- net /CM5_CONN_B/USB2_RP2350.USB_N: track 54.6 -> 53.0 mm
- net /Power Supply/VSYS: track 21.8 -> 20.3 mm
- net 3V3: track 217.6 -> 216.8 mm
- net /I2C2.I2C_SCL: track 201.1 -> 200.5 mm
- net /CONTROLLER/L_DPAD_LEFT: track 73.3 -> 72.7 mm
- net Net-(L2--): track 13.0 -> 12.5 mm
- net /CONTROLLER/L_L2_TRIG: track 70.7 -> 70.1 mm
- added copper zone on B.Cu, net GND
- added copper zone on In2.Cu, net GND
