File: hardware/Rev1_00-0a/Consolation_Kicad/TFT CONN.kicad_sch (KiCad schematic)
At the start: 35 parts, among them J3 62684-402100ALF, U11 AP22913W6-7, U26 TPS61169DCKR

Commit message: Add teardrops, clean ERC and DRC check. Review design rules Update fill zones Add stitching vias
Changed lines of the file:
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@@
 	(title_block
 		(title "Consolation [Console Emulation]")
-		(date "2026-10-26")
+		(date "2026-10-27")
 		(rev "1.00-0A")
 		(comment 1 "Jean-Francois Bilodeau")
@@
 		(comment 6 "Jean-Francois Bilodeau")
 		(comment 7 "Not applicable")
-		(comment 8 "In Design")
+		(comment 8 "In DFM Review")
 		(comment 9 "Consolation_1.00-0A_BOM")
 	)
@@
 	)
 	(junction
-		(at 92.075 189.865)
-		(diameter 0)
-		(color 0 0 0 0)
-	)
-	(junction
 		(at 255.27 113.03)
 		(diameter 0)
@@
 	)
 	(junction
-		(at 160.655 93.98)
+		(at 105.41 189.865)
 		(diameter 0)
 		(color 0 0 0 0)
 	)
 	(junction
-		(at 184.15 40.64)
+		(at 160.655 93.98)
 		(diameter 0)
 		(color 0 0 0 0)
 	)
 	(junction
-		(at 184.15 68.58)
+		(at 184.15 40.64)
 		(diameter 0)
 		(color 0 0 0 0)
 	)
 	(junction
-		(at 105.41 189.23)
+		(at 184.15 68.58)
 		(diameter 0)
 		(color 0 0 0 0)
@@
 	)
 	(junction
+		(at 92.075 189.865)
+		(diameter 0)
+		(color 0 0 0 0)
+	)
+	(junction
 		(at 107.315 101.6)
 		(diameter 0)
@@
 	(wire
 		(pts
-			(xy 105.41 189.23) (xy 105.41 190.5)
-		)
-		(stroke
-			(width 0)
-			(type default)
-		)
-	)
-	(wire
-		(pts
 			(xy 175.26 109.22) (xy 221.615 109.22)
 		)
@@
 	(wire
 		(pts
-			(xy 105.41 188.087) (xy 105.41 189.23)
-		)
-		(stroke
-			(width 0)
-			(type default)
-		)
-	)
-	(wire
-		(pts
 			(xy 146.685 48.26) (xy 184.15 48.26)
 		)
@@
 	(wire
 		(pts
-			(xy 146.685 116.205) (xy 146.685 118.11)
+			(xy 146.685 116.84) (xy 146.685 118.11)
 		)
 		(stroke
@@
 	(wire
 		(pts
-			(xy 92.075 188.087) (xy 92.075 189.865)
+			(xy 180.975 81.28) (xy 180.975 88.265)
 		)
 		(stroke
@@
 	(wire
 		(pts
-			(xy 180.975 81.28) (xy 180.975 88.265)
+			(xy 160.655 95.25) (xy 160.655 93.98)
 		)
 		(stroke
@@
 	(wire
 		(pts
-			(xy 160.655 95.25) (xy 160.655 93.98)
+			(xy 146.685 43.18) (xy 184.15 43.18)
 		)
 		(stroke
@@
 	(wire
 		(pts
-			(xy 146.685 43.18) (xy 184.15 43.18)
+			(xy 255.27 110.49) (xy 255.27 113.03)
 		)
 		(stroke
@@
 	(wire
 		(pts
-			(xy 255.27 110.49) (xy 255.27 113.03)
+			(xy 255.27 115.57) (xy 257.81 115.57)
 		)
 		(stroke
@@
 	(wire
 		(pts
-			(xy 255.27 115.57) (xy 257.81 115.57)
+			(xy 105.41 189.865) (xy 105.41 190.5)
 		)
 		(stroke
@@
 	(wire
 		(pts
-			(xy 85.09 188.087) (xy 85.09 189.865)
-		)
-		(stroke
-			(width 0)
-			(type default)
-		)
-	)
-	(wire
-		(pts
 			(xy 201.93 62.23) (xy 257.81 62.23)
 		)
@@
 	(wire
 		(pts
+			(xy 112.395 188.595) (xy 112.395 189.865)
+		)
+		(stroke
+			(width 0)
+			(type default)
+		)
+	)
+	(wire
+		(pts
 			(xy 141.605 93.98) (xy 144.78 93.98)
 		)
@@
 	(wire
 		(pts
+			(xy 92.075 188.595) (xy 92.075 189.865)
+		)
+		(stroke
+			(width 0)
+			(type default)
+		)
+	)
+	(wire
+		(pts
 			(xy 153.67 95.25) (xy 153.67 93.98)
 		)
@@
 	(wire
 		(pts
-			(xy 105.41 189.23) (xy 112.395 189.23)
+			(xy 105.41 189.865) (xy 112.395 189.865)
 		)
 		(stroke
@@
 		)
 	)
+	(wire
+		(pts
+			(xy 85.09 188.595) (xy 85.09 189.865)
+		)
+		(stroke
+			(width 0)
+			(type default)
+		)
+	)
 	(bus
 		(pts
@@
 	(wire
 		(pts
-			(xy 112.395 188.087) (xy 112.395 189.23)
+			(xy 105.41 188.595) (xy 105.41 189.865)
 		)
 		(stroke
@@
 	(wire
 		(pts
-			(xy 153.67 116.205) (xy 153.67 118.11)
+			(xy 153.67 116.84) (xy 153.67 118.11)
 		)
 		(stroke
@@
 	(symbol
 		(lib_id "KicadCompDb:Resistors/RES_SMT_00007")
-		(at 153.67 114.935 90)
+		(at 153.67 115.57 90)
 		(unit 1)
 		(body_style 1)
@@
 		(dnp yes)
 		(property "Reference" "R213"
-			(at 153.035 111.633 90)
+			(at 153.035 112.268 90)
 			(show_name no)
 			(do_not_autoplace no)
@@
 		)
 		(property "Value" "1R5"
-			(at 153.035 113.411 90)
+			(at 153.035 114.046 90)
 			(show_name no)
 			(do_not_autoplace no)
@@
 		)
 		(property "Footprint" "footprint:RES_0603"
-			(at 175.768 114.427 0)
+			(at 175.768 115.062 0)
 			(hide yes)
 			(show_name no)
@@
 		)
 		(property "Datasheet" "https://www.yageogroup.com/content/datasheet/asset/file/PYU-RC_GROUP_51_ROHS_L"
-			(at 153.67 114.935 0)
+			(at 153.67 115.57 0)
 			(hide yes)
 			(show_name no)
@@
 		)
 		(property "Description" "RES 1.5 OHM 1% 1/10W 0603"
-			(at 163.576 113.157 0)
+			(at 163.576 113.792 0)
 			(hide yes)
 			(show_name no)
@@
 		)
 		(property "Tolerance" "1%"
-			(at 156.972 112.141 0)
+			(at 156.972 112.776 0)
 			(hide yes)
 			(show_name no)
@@
 		)
 		(property "Power" "1/10W"
-			(at 151.765 114.5539 90)
+			(at 151.765 115.1889 90)
 			(hide yes)
 			(show_name no)
@@
 		)
 		(property "Package" "0603"
-			(at 153.035 115.189 90)
+			(at 153.035 115.824 90)
 			(show_name no)
 			(do_not_autoplace no)
@@
 		)
 		(property "Manufacturer" "YAGEO"
-			(at 171.958 114.681 0)
+			(at 171.958 115.316 0)
 			(hide yes)
 			(show_name no)
@@
 		)
 		(property "Manufacturer Part Number" "RC0603FR-131R5L"
-			(at 161.544 114.681 0)
+			(at 161.544 115.316 0)
 			(hide yes)
 			(show_name no)
@@
 		)
 		(property "Distributor" "DigiKey"
-			(at 159.512 114.935 0)
+			(at 159.512 115.57 0)
 			(hide yes)
 			(show_name no)
@@
 		)
 		(property "Distributor Part Number" "13-RC0603FR-131R5LCT-ND"
-			(at 165.862 114.173 0)
+			(at 165.862 114.808 0)
 			(hide yes)
 			(show_name no)
@@
 		)
 		(property "Temperature Coefficient" "±200ppm/°C"
-			(at 153.67 114.935 0)
+			(at 153.67 115.57 0)
 			(hide yes)
 			(show_name no)
@@
 		)
 		(property "Operating Temperature" "-55°C ~ 155°C"
-			(at 178.054 114.173 0)
+			(at 178.054 114.808 0)
 			(hide yes)
 			(show_name no)
@@
 		)
 		(property "Type" "RES SMT"
-			(at 153.67 114.935 0)
+			(at 153.67 115.57 0)
 			(hide yes)
 			(show_name yes)
@@
 		)
 		(property "Dimensions" "1.60mm x 0.80mm"
-			(at 153.67 114.935 0)
+			(at 153.67 115.57 0)
 			(hide yes)
 			(show_name yes)
@@
 	(symbol
 		(lib_id "KicadCompDb:Resistors/RES_SMT_00007")
-		(at 146.685 114.935 90)
+		(at 146.685 115.57 90)
 		(unit 1)
 		(body_style 1)
@@
 		(dnp no)
 		(property "Reference" "R210"
-			(at 146.05 111.633 90)
+			(at 146.05 112.268 90)
 			(show_name no)
 			(do_not_autoplace no)
@@
 		)
 		(property "Value" "1R5"
-			(at 146.05 113.411 90)
+			(at 146.05 114.046 90)
 			(show_name no)
 			(do_not_autoplace no)
@@
 		)
 		(property "Footprint" "footprint:RES_0603"
-			(at 168.783 114.427 0)
+			(at 168.783 115.062 0)
 			(hide yes)
 			(show_name no)
@@
 		)
 		(property "Datasheet" "https://www.yageogroup.com/content/datasheet/asset/file/PYU-RC_GROUP_51_ROHS_L"
-			(at 146.685 114.935 0)
+			(at 146.685 115.57 0)
 			(hide yes)
 			(show_name no)
@@
 		)
 		(property "Description" "RES 1.5 OHM 1% 1/10W 0603"
-			(at 156.591 113.157 0)
+			(at 156.591 113.792 0)
 			(hide yes)
 			(show_name no)
@@
 		)
 		(property "Tolerance" "1%"
-			(at 149.987 112.141 0)
+			(at 149.987 112.776 0)
 			(hide yes)
 			(show_name no)
@@
 		)
 		(property "Power" "1/10W"
-			(at 144.78 114.5539 90)
+			(at 144.78 115.1889 90)
 			(hide yes)
 			(show_name no)
@@
 		)
 		(property "Package" "0603"
-			(at 146.05 115.189 90)
+			(at 146.05 115.824 90)
 			(show_name no)
 			(do_not_autoplace no)
@@
 		)
 		(property "Manufacturer" "YAGEO"
-			(at 164.973 114.681 0)
+			(at 164.973 115.316 0)
 			(hide yes)
 			(show_name no)
@@
 		)
 		(property "Manufacturer Part Number" "RC0603FR-131R5L"
-			(at 154.559 114.681 0)
+			(at 154.559 115.316 0)
 			(hide yes)
 			(show_name no)
@@
 		)
 		(property "Distributor" "DigiKey"
-			(at 152.527 114.935 0)
+			(at 152.527 115.57 0)
 			(hide yes)
 			(show_name no)
@@
 		)
 		(property "Distributor Part Number" "13-RC0603FR-131R5LCT-ND"
-			(at 158.877 114.173 0)
+			(at 158.877 114.808 0)
 			(hide yes)
 			(show_name no)
@@
 		)
 		(property "Temperature Coefficient" "±200ppm/°C"
-			(at 146.685 114.935 0)
+			(at 146.685 115.57 0)
 			(hide yes)
 			(show_name no)
@@
 		)
 		(property "Operating Temperature" "-55°C ~ 155°C"
-			(at 171.069 114.173 0)
+			(at 171.069 114.808 0)
 			(hide yes)
 			(show_name no)
@@
 		)
 		(property "Type" "RES SMT"
-			(at 146.685 114.935 0)
+			(at 146.685 115.57 0)
 			(hide yes)
 			(show_name yes)
@@
 		)
 		(property "Dimensions" "1.60mm x 0.80mm"
-			(at 146.685 114.935 0)
+			(at 146.685 115.57 0)
 			(hide yes)
 			(show_name yes)
