File: hardware/Rev1_00-0a/Consolation_Kicad/CONTROLLER.kicad_sch (KiCad schematic)
At the start: 83 parts, among them J11 5051102291, J13 5051102291, J14 61300311121, J15 61300311121, Q18 SSM3K56FS,LF, U2 RP2350A, U8 GD25Q32CWIGR, Y1 12MHz 10pF

Commit message: Add teardrops, clean ERC and DRC check. Review design rules Update fill zones Add stitching vias
Parts:
- R204: Manufacturer Part Number RC0402FR-071KL -> RC0402JR-070RL
Changed lines of the file:
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@@
 	(title_block
 		(title "Consolation [Console Emulation]")
-		(date "2026-10-26")
+		(date "2026-10-27")
 		(rev "1.00-0A")
 		(comment 1 "Jean-Francois Bilodeau")
@@
 		(comment 6 "Jean-Francois Bilodeau")
 		(comment 7 "Not applicable")
-		(comment 8 "In Design")
+		(comment 8 "In DFM Review")
 		(comment 9 "Consolation_1.00-0A_BOM")
 	)
@@
 			)
 		)
-		(property "Manufacturer Part Number" "RC0402FR-071KL"
+		(property "Manufacturer Part Number" "RC0402JR-070RL"
 			(at 122.174 67.564 0)
 			(hide yes)

Commit message: Add preliminary manufacturing files for Consolation Review pinout & design notes
Parts:
- removed C148, C153: 1u, footprint:CAP_NONPOL_0805, symbol KicadCompDb:Capacitors/CAP_CER_SMT_00002
- removed R12: 100R, footprint:RES_0402, symbol KicadCompDb:Resistors/RES_SMT_00035
- removed R192, R193, R194, R195: 10K, footprint:RES_0402, symbol KicadCompDb:Resistors/RES_SMT_00013
- added C148, C153: 4.7u, footprint:CAP_NONPOL_0805, symbol KicadCompDb:Capacitors/CAP_CER_SMT_00017
- added R12: 22R, footprint:RES_0402, symbol KicadCompDb:Resistors/RES_SMT_00015
Connections:
- net 3V3: now also R12.1
- net GND: now also C148.2, C153.2
- net L_HOME: now also R185.1, U2.10 (GPIO7); no longer U2.43 (GPIO29_ADC3)
- net L_L1_TRIG: now also R189.1, U2.31 (GPIO19); no longer U2.41 (GPIO27_ADC1)
- net L_L2_TRIG: now also R181.1, U2.9 (GPIO6); no longer U2.42 (GPIO28_ADC2)
- net L_START: now also R191.1, U2.28 (GPIO17); no longer U2.40 (GPIO26_ADC0)
- net L_THUMBST_X: now also U2.40 (GPIO26_ADC0); no longer R191.1, U2.28 (GPIO17)
- net L_THUMBST_Y: now also U2.41 (GPIO27_ADC1); no longer R189.1, U2.31 (GPIO19)
- net R_THUMBST_X: now also U2.42 (GPIO28_ADC2); no longer R181.1, U2.9 (GPIO6)
- net R_THUMBST_Y: now also U2.43 (GPIO29_ADC3); no longer R185.1, U2.10 (GPIO7)
- net at C149.2, U2.44 (ADC_AVDD): now also C148.1, R12.2
- net at C152.2, R134.2, U2.46 (VREG_AVDD): now also C153.1
Other:
- note added: "SW-trig'd HW reset (CM5)"
- note removed: "SW reset (CM5)"
- moved on the sheet: R284

Commit message: Work on DFM, Pick N Place file accuracy, BOM accuracy Generating output files regularly through incremental updates
Parts:
- TP34, TP35, TP36: now left out of the parts list
Changed lines of the file:
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@@
 		(body_style 1)
 		(exclude_from_sim no)
-		(in_bom yes)
+		(in_bom no)
 		(on_board yes)
-		(in_pos_files yes)
+		(in_pos_files no)
 		(dnp no)
 		(property "Reference" "TP34"
@@
 		(body_style 1)
 		(exclude_from_sim no)
-		(in_bom yes)
+		(in_bom no)
 		(on_board yes)
-		(in_pos_files yes)
+		(in_pos_files no)
 		(dnp no)
 		(property "Reference" "TP36"
@@
 		(body_style 1)
 		(exclude_from_sim no)
-		(in_bom yes)
+		(in_bom no)
 		(on_board yes)
-		(in_pos_files yes)
+		(in_pos_files no)
 		(dnp no)
 		(property "Reference" "TP35"
