File: hardware/Rev1_00-0a/Consolation_Kicad/HDMI.kicad_sch (KiCad schematic)
At the start: 10 parts, among them J6 2086581001, U18 AP22913W6-7

Commit message: Preliminary routing (DiffPairs, Power planes) in progress Slight changes to schematics to accommodate routing
Connections:
- net 5V0_CB renamed 5V0
Changed lines of the file:
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@@
 	(title_block
 		(title "Consolation [Console Emulation]")
-		(date "2026-09-20")
+		(date "2026-10-12")
 		(rev "1.00-0A")
 		(comment 1 "Jean-Francois Bilodeau")
@@
 			(justify left bottom)
 		)
-		(property "Net Class" "DP_100R"
+		(property "Netclass" "DP_100R"
 			(at 139.954 51.181 0)
 			(show_name no)
@@
 			(justify left bottom)
 		)
-		(property "Net Class" "DP_100R"
+		(property "Netclass" "DP_100R"
 			(at 139.954 56.261 0)
 			(show_name no)
@@
 			(justify left bottom)
 		)
-		(property "Net Class" "DP_100R"
+		(property "Netclass" "DP_100R"
 			(at 139.954 79.629 0)
 			(show_name no)
@@
 			(justify left bottom)
 		)
-		(property "Net Class" "DP_100R"
+		(property "Netclass" "DP_100R"
 			(at 139.954 58.801 0)
 			(show_name no)
@@
 			(justify left bottom)
 		)
-		(property "Net Class" "DP_100R"
+		(property "Netclass" "DP_100R"
 			(at 139.954 61.341 0)
 			(show_name no)
@@
 			(justify left bottom)
 		)
-		(property "Net Class" "DP_100R"
+		(property "Netclass" "DP_100R"
 			(at 139.954 48.641 0)
 			(show_name no)
@@
 			(justify left bottom)
 		)
-		(property "Net Class" "DP_100R"
+		(property "Netclass" "DP_100R"
 			(at 139.954 82.169 0)
 			(show_name no)
@@
 			(justify left bottom)
 		)
-		(property "Net Class" "DP_100R"
+		(property "Netclass" "DP_100R"
 			(at 139.954 53.721 0)
 			(show_name no)
@@
 			)
 		)
-		(property "Value" "5V0_CB"
+		(property "Value" "5V0"
 			(at 128.27 104.775 0)
 			(show_name no)

Commit message: Work on DFM, Pick N Place file accuracy, BOM accuracy Generating output files regularly through incremental updates
Parts:
- TP48: now left out of the parts list
Changed lines of the file:
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@@
 		(body_style 1)
 		(exclude_from_sim no)
-		(in_bom yes)
+		(in_bom no)
 		(on_board yes)
-		(in_pos_files yes)
+		(in_pos_files no)
 		(dnp no)
 		(property "Reference" "TP48"
