File: hardware/Rev1_00-0a/Consolation_Kicad/Power Supply.kicad_sch (KiCad schematic)
At the start: 49 parts, among them Q1 SSM3K56FS,LF, Q3 SSM3K56FS,LF, U10 TPS62826DMQR, U7 TPS79901DRVR, U9 TPS61230ARNSR

Commit message: Add preliminary manufacturing files for Consolation Review pinout & design notes
Parts:
- removed C28, C36, C42: 1u, footprint:CAP_NONPOL_0805, symbol KicadCompDb:Capacitors/CAP_CER_SMT_00002
- removed C33: 100p, footprint:CAP_NONPOL_0402, symbol KicadCompDb:Capacitors/CAP_CER_SMT_00007
- added C28, C36, C42: 22u, footprint:CAP_NONPOL_0805, symbol KicadCompDb:Capacitors/CAP_CER_SMT_00011
- added C33: 120p, footprint:CAP_NONPOL_0402, symbol KicadCompDb:Capacitors/CAP_CER_SMT_00021
Connections:
- net 1V8: now also R164.2, C42.2; no longer R33.2
- net 3V3: now also C33.2, C36.2
- net 5V0: now also C28.2
- net GND: now also R33.1, C28.1, C36.1, C42.1; no longer R164.1
- net at C39.1, U7.2 (FB): now also R164.1, R33.2; no longer R164.2, R33.1
- net at R30.1, R31.2, U10.3 (FB): now also C33.1

Commit message: Work on DFM, Pick N Place file accuracy, BOM accuracy Generating output files regularly through incremental updates
Parts:
- TP10, TP11, TP12, TP13, TP14, TP50, TP51, TP9: now left out of the parts list
Changed lines of the file:
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@@
 		(body_style 1)
 		(exclude_from_sim no)
-		(in_bom yes)
+		(in_bom no)
 		(on_board yes)
-		(in_pos_files yes)
+		(in_pos_files no)
 		(dnp no)
 		(property "Reference" "TP13"
@@
 		(body_style 1)
 		(exclude_from_sim no)
-		(in_bom yes)
+		(in_bom no)
 		(on_board yes)
-		(in_pos_files yes)
+		(in_pos_files no)
 		(dnp no)
 		(property "Reference" "TP14"
@@
 		(body_style 1)
 		(exclude_from_sim no)
-		(in_bom yes)
+		(in_bom no)
 		(on_board yes)
-		(in_pos_files yes)
+		(in_pos_files no)
 		(dnp no)
 		(property "Reference" "TP12"
@@
 		(body_style 1)
 		(exclude_from_sim no)
-		(in_bom yes)
+		(in_bom no)
 		(on_board yes)
-		(in_pos_files yes)
+		(in_pos_files no)
 		(dnp no)
 		(property "Reference" "TP51"
@@
 		(body_style 1)
 		(exclude_from_sim no)
-		(in_bom yes)
+		(in_bom no)
 		(on_board yes)
-		(in_pos_files yes)
+		(in_pos_files no)
 		(dnp no)
 		(property "Reference" "TP11"
@@
 		(body_style 1)
 		(exclude_from_sim no)
-		(in_bom yes)
+		(in_bom no)
 		(on_board yes)
-		(in_pos_files yes)
+		(in_pos_files no)
 		(dnp no)
 		(property "Reference" "TP50"
@@
 		(body_style 1)
 		(exclude_from_sim no)
-		(in_bom yes)
+		(in_bom no)
 		(on_board yes)
-		(in_pos_files yes)
+		(in_pos_files no)
 		(dnp no)
 		(property "Reference" "TP9"
@@
 		(body_style 1)
 		(exclude_from_sim no)
-		(in_bom yes)
+		(in_bom no)
 		(on_board yes)
-		(in_pos_files yes)
+		(in_pos_files no)
 		(dnp no)
 		(property "Reference" "TP10"
