File: hardware/Rev1_00-0a/Consolation_Kicad/RESET SUPERVISOR.kicad_sch (KiCad schematic)
At the start: 36 parts, among them Q7 SSM3K56FS,LF, Q8 SSM3K56FS,LF, Q9 SSM3K56FS,LF, U30 STM6710DWB6F, U31 SN74LVC1G125DBVR, U32 SN74HCS365QPWRQ1

Commit message: Add teardrops, clean ERC and DRC check. Review design rules Update fill zones Add stitching vias
Parts:
- R169, R170, R172, R206, R207, R214, R215: Manufacturer Part Number RC0402FR-071KL -> RC0402JR-070RL
Changed lines of the file:
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@@
 	(title_block
 		(title "Consolation [Console Emulation]")
-		(date "2026-10-26")
+		(date "2026-10-27")
 		(rev "1.00-0A")
 		(comment 1 "Jean-Francois Bilodeau")
@@
 		(comment 6 "Jean-Francois Bilodeau")
 		(comment 7 "Not applicable")
-		(comment 8 "In Design")
+		(comment 8 "In DFM Review")
 		(comment 9 "Consolation_1.00-0A_BOM")
 	)
@@
 		)
 	)
-	(netclass_flag ""
-		(length 2.54)
-		(shape round)
-		(at 145.415 62.23 0)
-		(fields_autoplaced yes)
-		(effects
-			(font
-				(size 1.27 1.27)
-			)
-			(justify left bottom)
-		)
-		(property "Netclass" "CRITICAL"
-			(at 146.1135 59.69 0)
-			(show_name no)
-			(do_not_autoplace no)
-			(effects
-				(font
-					(size 1.27 1.27)
-					(color 255 0 0 1)
-				)
-				(justify left)
-			)
-		)
-		(property "Component Class" ""
-			(at 90.805 23.495 0)
-			(show_name no)
-			(do_not_autoplace no)
-			(effects
-				(font
-					(size 1.27 1.27)
-					(italic yes)
-				)
-			)
-		)
-	)
 	(symbol
 		(lib_id "KiCad_Pwr_Symbols:GND")
@@
 			)
 		)
-		(property "Manufacturer Part Number" "RC0402FR-071KL"
+		(property "Manufacturer Part Number" "RC0402JR-070RL"
 			(at 60.579 77.851 0)
 			(hide yes)
@@
 			)
 		)
-		(property "Manufacturer Part Number" "RC0402FR-071KL"
+		(property "Manufacturer Part Number" "RC0402JR-070RL"
 			(at 99.949 58.801 0)
 			(hide yes)
@@
 			)
 		)
-		(property "Manufacturer Part Number" "RC0402FR-071KL"
+		(property "Manufacturer Part Number" "RC0402JR-070RL"
 			(at 74.549 77.851 0)
 			(hide yes)
@@
 			)
 		)
-		(property "Manufacturer Part Number" "RC0402FR-071KL"
+		(property "Manufacturer Part Number" "RC0402JR-070RL"
 			(at 102.489 77.851 0)
 			(hide yes)
@@
 			)
 		)
-		(property "Manufacturer Part Number" "RC0402FR-071KL"
+		(property "Manufacturer Part Number" "RC0402JR-070RL"
 			(at 72.009 58.801 0)
 			(hide yes)
@@
 			)
 		)
-		(property "Manufacturer Part Number" "RC0402FR-071KL"
+		(property "Manufacturer Part Number" "RC0402JR-070RL"
 			(at 85.979 58.801 0)
 			(hide yes)
@@
 			)
 		)
-		(property "Manufacturer Part Number" "RC0402FR-071KL"
+		(property "Manufacturer Part Number" "RC0402JR-070RL"
 			(at 88.519 77.851 0)
 			(hide yes)

Commit message: Add preliminary manufacturing files for Consolation Review pinout & design notes
Other:
- note added: "Peripherals reset"
- note added: "Power Good"
Changed lines of the file:
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@@
 	(title_block
 		(title "Consolation [Console Emulation]")
-		(date "2026-10-27")
+		(date "2026-10-31")
 		(rev "1.00-0A")
 		(comment 1 "Jean-Francois Bilodeau")
@@
 			)
 		)
+	)
+	(text "Power Good"
+		(exclude_from_sim no)
+		(at 112.268 78.486 0)
+		(effects
+			(font
+				(size 1.27 1.27)
+				(color 255 153 0 1)
+			)
+		)
+	)
+	(text "Peripherals reset"
+		(exclude_from_sim no)
+		(at 198.628 110.998 0)
+		(effects
+			(font
+				(size 1.27 1.27)
+				(color 255 153 0 1)
+			)
+		)

Commit message: Work on DFM, Pick N Place file accuracy, BOM accuracy Generating output files regularly through incremental updates
Parts:
- TP15, TP16, TP17: now left out of the parts list
Changed lines of the file:
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@@
 		(body_style 1)
 		(exclude_from_sim no)
-		(in_bom yes)
+		(in_bom no)
 		(on_board yes)
-		(in_pos_files yes)
+		(in_pos_files no)
 		(dnp no)
 		(property "Reference" "TP16"
@@
 		(body_style 1)
 		(exclude_from_sim no)
-		(in_bom yes)
+		(in_bom no)
 		(on_board yes)
-		(in_pos_files yes)
+		(in_pos_files no)
 		(dnp no)
 		(property "Reference" "TP17"
@@
 		(body_style 1)
 		(exclude_from_sim no)
-		(in_bom yes)
+		(in_bom no)
 		(on_board yes)
-		(in_pos_files yes)
+		(in_pos_files no)
 		(dnp no)
 		(property "Reference" "TP15"
