File: hardware/Rev1_00-0a/Consolation_Kicad/RPI_CM5_B.kicad_sch (KiCad schematic)
At the start: 13 parts, among them J12 RPI_CMx_B, J18 61300411121

Commit message: Work on DFM, Pick N Place file accuracy, BOM accuracy Generating output files regularly through incremental updates
Parts:
- J12: value RPI_CMx_B -> DF40HC(3.0)-100DS-0.4V
- TP23: now left out of the parts list
Changed lines of the file:
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@@
 			)
 		)
-		(property "Value" "RPI_CMx_B"
-			(at 174.752 21.336 0)
+		(property "Value" "DF40HC(3.0)-100DS-0.4V"
+			(at 166.878 21.336 0)
 			(show_name no)
 			(do_not_autoplace no)
@@
 		(body_style 1)
 		(exclude_from_sim no)
-		(in_bom yes)
+		(in_bom no)
 		(on_board yes)
-		(in_pos_files yes)
+		(in_pos_files no)
 		(dnp no)
 		(property "Reference" "TP23"
