File: hardware/Rev1_00-0a/Consolation_Kicad/SD_CARD.kicad_sch (KiCad schematic)
At the start: 18 parts, among them J8 DM3AT-SF-PEJM5, Q23 SSM3K56FS,LF, Q24 SSM3K56FS,LF, Q25 SSM3K56FS,LF, U6 AP22913W6-7

Commit message: Add preliminary manufacturing files for Consolation Review pinout & design notes
Parts:
- added D31: ESD7351HT1G, footprint:SOD-323, symbol KicadCompDb:ESD Diodes/ESD_DIODE_00006
Connections:
- net GND: now also D31.2 (A)
- net SD_VDD: now also D31.1 (K)

Commit message: Work on DFM, Pick N Place file accuracy, BOM accuracy Generating output files regularly through incremental updates
Parts:
- TP18, TP19: now left out of the parts list
Changed lines of the file:
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@@
 		(body_style 1)
 		(exclude_from_sim no)
-		(in_bom yes)
+		(in_bom no)
 		(on_board yes)
-		(in_pos_files yes)
+		(in_pos_files no)
 		(dnp no)
 		(property "Reference" "TP19"
@@
 		(body_style 1)
 		(exclude_from_sim no)
-		(in_bom yes)
+		(in_bom no)
 		(on_board yes)
-		(in_pos_files yes)
+		(in_pos_files no)
 		(dnp no)
 		(property "Reference" "TP18"
